Commit message: version working on ros with velocity control on wheels

File: locomotion_framework/xbot/robot_class_xbot/include/configs/urdf/centauro_full.urdf (robot description, URDF)
Before this commit: robot centauro, 44 links, 43 joints
Joints:
- joint j_arm1_8: axis 1 0 0 -> (none); limit lower=0.0 upper=0 effort=0 velocity=0 -> (none); type revolute -> fixed
- joint j_arm2_8: axis 1 0 0 -> (none); limit lower=0.0 upper=0 effort=0 velocity=0 -> (none); type revolute -> fixed
