Commit message: xbot working with velocity

File: locomotion_framework/xbot/robot_class_xbot/include/configs/urdf/centauro_lower_body.urdf (robot description, URDF)
Before this commit: robot centauro, 26 links, 25 joints
Links:
- added link imu_link, mass 0.0
Joints:
- added joint imu_joint: type fixed, parent pelvis, child imu_link, origin xyz=0.0 0.0 0.0 rpy=0.0 0.0 0.0
- joint hip_yaw_1: limit lower=-0.78539816 upper=2.35619449 effort=304 velocity=8.8 -> lower=-1.13446401 upper=2.70526034 effort=304 velocity=8.8; origin xyz=0.225 0.125 0.11 rpy=3.14159265359 0.0 0.50709869865 -> xyz=0.25 0.125 -0.0566 rpy=3.14159265359 0.0 0.50709869865
- joint hip_yaw_2: limit lower=-2.35619449 upper=0.78539816 effort=304 velocity=8.8 -> lower=-2.70526034 upper=1.13446401 effort=304 velocity=8.8; origin xyz=0.225 -0.125 0.11 rpy=3.14159265359 0.0 -0.50709869865 -> xyz=0.25 -0.125 -0.0566 rpy=3.14159265359 0.0 -0.50709869865
- joint hip_yaw_3: limit lower=-2.35619449 upper=0.78539816 effort=304 velocity=8.8 -> lower=-2.70526034 upper=1.13446401 effort=304 velocity=8.8; origin xyz=-0.225 0.125 0.11 rpy=3.14159265359 0.0 2.63449395494 -> xyz=-0.25 0.125 -0.0566 rpy=3.14159265359 0.0 2.63449395494
- joint hip_yaw_4: limit lower=-0.78539816 upper=2.35619449 effort=304 velocity=8.8 -> lower=-1.13446401 upper=2.70526034 effort=304 velocity=8.8; origin xyz=-0.225 -0.125 0.11 rpy=3.14159265359 0.0 3.64869135224 -> xyz=-0.25 -0.125 -0.0566 rpy=3.14159265359 0.0 3.64869135224
- joint reference: origin xyz=0.0 0.0 0.759 -> xyz=0.0 0.0 0.9256

File: locomotion_framework/xbot/robot_class_xbot/include/configs/urdf/centauro_static.urdf (robot description, URDF)
Before this commit: robot centauro, 44 links, 43 joints
Links:
- removed link arm1_1
- removed link arm1_2
- removed link arm1_3
- removed link arm1_4
- removed link arm1_5
- removed link arm1_6
- removed link arm1_7
- removed link arm1_8
- removed link arm2_1
- removed link arm2_2
- removed link arm2_3
- removed link arm2_4
- removed link arm2_5
- removed link arm2_6
- removed link arm2_7
- removed link arm2_8
- removed link torso_2
Joints:
- removed joint j_arm1_1
- removed joint j_arm1_2
- removed joint j_arm1_3
- removed joint j_arm1_4
- removed joint j_arm1_5
- removed joint j_arm1_6
- removed joint j_arm1_7
- removed joint j_arm1_8
- removed joint j_arm2_1
- removed joint j_arm2_2
- removed joint j_arm2_3
- removed joint j_arm2_4
- removed joint j_arm2_5
- removed joint j_arm2_6
- removed joint j_arm2_7
- removed joint j_arm2_8
- removed joint torso_yaw
- joint reference: type floating -> fixed
