Commit message: experiments xbot api changes

File: locomotion_framework/xbot/robot_class_xbot/include/configs/urdf/centauro_v2.urdf (robot description, URDF)
Before this commit: robot centauro, 57 links, 56 joints
Links:
- removed link fl_foot_ft
- removed link foot_fl
- removed link foot_fr
- removed link foot_hl
- removed link foot_hr
- removed link fr_foot_ft
- removed link ft_arm1
- removed link ft_arm2
- removed link hl_foot_ft
- removed link hr_foot_ft
- removed link neck_1
- removed link neck_2
- removed link neck_3
Joints:
- removed joint j_fl_foot_ft
- removed joint j_foot_fl
- removed joint j_foot_fr
- removed joint j_foot_hl
- removed joint j_foot_hr
- removed joint j_fr_foot_ft
- removed joint j_ft_arm1
- removed joint j_ft_arm2
- removed joint j_hl_foot_ft
- removed joint j_hr_foot_ft
- removed joint neck_pitch
- removed joint neck_velodyne
- removed joint neck_yaw
- joint j_arm1_2: limit lower=-3.49 upper=-0.25 effort=147 velocity=5.7 -> lower=-3.49 upper=0 effort=147 velocity=5.7
- joint j_arm1_8: limit lower=0.0 upper=0 effort=0 velocity=0 -> (none)
- joint j_arm2_2: limit lower=0.25 upper=3.49 effort=147 velocity=5.7 -> lower=0 upper=3.49 effort=147 velocity=5.7
- joint j_arm2_8: limit lower=0.0 upper=0 effort=0 velocity=0 -> (none)
- joint j_wheel_1: limit lower=-1000000000000000 upper=1000000000000000 effort=35 velocity=20.0 -> effort=35 velocity=20.0; origin xyz=0.0 0.00085 0.235 rpy=1.57079632679 0.0 0.0 -> xyz=0.0 0.00085 0.237350 rpy=1.57079632679 0.0 3.14159265359
- joint j_wheel_2: limit lower=-1000000000000000 upper=1000000000000000 effort=35 velocity=20.0 -> effort=35 velocity=20.0; origin xyz=0.0 0.00085 0.235 rpy=1.57079632679 0.0 0.0 -> xyz=0.0 0.00085 0.237350 rpy=1.57079632679 0.0 3.14159265359
- joint j_wheel_3: limit lower=-1000000000000000 upper=1000000000000000 effort=35 velocity=20.0 -> effort=35 velocity=20.0; origin xyz=0.0 0.00085 0.235 rpy=1.57079632679 0.0 0.0 -> xyz=0.0 0.00085 0.237350 rpy=1.57079632679 0.0 3.14159265359
- joint j_wheel_4: limit lower=-1000000000000000 upper=1000000000000000 effort=35 velocity=20.0 -> effort=35 velocity=20.0; origin xyz=0.0 0.00085 0.235 rpy=1.57079632679 0.0 0.0 -> xyz=0.0 0.00085 0.237350 rpy=1.57079632679 0.0 3.14159265359
- joint reference: origin xyz=0.0 0.0 0.9256 -> xyz=0.0 0.0 0.92795000
