Commit message: Add flag to cmake files to find third party libraries
Add getErrorFull methods

File: locomotion_framework/xbot/robot_class_xbot/include/configs/urdf/centauro.urdf (robot description, URDF)
Before this commit: robot centauro, 48 links, 47 joints
Links:
- removed link foot_fl
- removed link foot_fr
- removed link foot_hl
- removed link foot_hr
- removed link imu_link
- added link pelvis_imu_link, mass 0.0
- link arm1_8: geometry collision mesh filename=package://centauro/centauro_urdf/meshes/convex_hull/link9.s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 scale=0.001 -0.001 -0.001
- link torso_2: mass 4.5494226 -> 6.1886404
Joints:
- removed joint imu_joint
- removed joint j_foot_fl
- removed joint j_foot_fr
- removed joint j_foot_hl
- removed joint j_foot_hr
- added joint pelvis_imu_joint: type fixed, parent pelvis, child pelvis_imu_link, origin xyz=0.0 0.0 0.0 rpy=0.0 0.0 0.0
- joint hip_yaw_1: limit lower=-0.78539816 upper=2.35619449 effort=304 velocity=8.8 -> lower=-1.13446401 upper=2.70526034 effort=304 velocity=8.8; origin xyz=0.225 0.125 0.11 rpy=3.14159265359 0.0 0.50709869865 -> xyz=0.25 0.125 -0.0566 rpy=3.14159265359 0.0 0.50709869865
- joint hip_yaw_2: limit lower=-2.35619449 upper=0.78539816 effort=304 velocity=8.8 -> lower=-2.70526034 upper=1.13446401 effort=304 velocity=8.8; origin xyz=0.225 -0.125 0.11 rpy=3.14159265359 0.0 -0.50709869865 -> xyz=0.25 -0.125 -0.0566 rpy=3.14159265359 0.0 -0.50709869865
- joint hip_yaw_3: limit lower=-2.35619449 upper=0.78539816 effort=304 velocity=8.8 -> lower=-2.70526034 upper=1.13446401 effort=304 velocity=8.8; origin xyz=-0.225 0.125 0.11 rpy=3.14159265359 0.0 2.63449395494 -> xyz=-0.25 0.125 -0.0566 rpy=3.14159265359 0.0 2.63449395494
- joint hip_yaw_4: limit lower=-0.78539816 upper=2.35619449 effort=304 velocity=8.8 -> lower=-1.13446401 upper=2.70526034 effort=304 velocity=8.8; origin xyz=-0.225 -0.125 0.11 rpy=3.14159265359 0.0 3.64869135224 -> xyz=-0.25 -0.125 -0.0566 rpy=3.14159265359 0.0 3.64869135224
- joint j_arm1_1: origin xyz=0.04576 0.169137 0.190626 rpy=0.0 0.0 -0.523602668986 -> xyz=0.04576 0.169137 0.116626 rpy=0.0 0.0 -0.523602668986
- joint j_arm1_8: axis 1 0 0 -> (none); limit lower=0.0 upper=0 effort=0 velocity=0 -> (none)
- joint j_arm2_1: origin xyz=0.04576 -0.169137 0.190626 rpy=0.0 0.0 0.523602668986 -> xyz=0.04576 -0.169137 0.116626 rpy=0.0 0.0 0.523602668986
- joint j_arm2_8: axis 1 0 0 -> (none); limit lower=0.0 upper=0 effort=0 velocity=0 -> (none)
- joint reference: origin xyz=0.0 0.0 0.759 -> xyz=0.0 0.0 0.9256
- joint torso_yaw: origin xyz=0.175 0.0 0.36 -> xyz=0.2 0.0 0.256

File: locomotion_framework/xbot/robot_class_xbot/include/configs/urdf/centauro_full.urdf (robot description, URDF)
Before this commit: robot centauro, 48 links, 47 joints
Links:
- removed link foot_fl
- removed link foot_fr
- removed link foot_hl
- removed link foot_hr
- link torso_2: mass 4.5494226 -> 6.1886404
Joints:
- removed joint j_foot_fl
- removed joint j_foot_fr
- removed joint j_foot_hl
- removed joint j_foot_hr
- joint hip_yaw_1: limit lower=-0.78539816 upper=2.35619449 effort=304 velocity=8.8 -> lower=-1.13446401 upper=2.70526034 effort=304 velocity=8.8; origin xyz=0.225 0.125 0.11 rpy=3.14159265359 0.0 0.50709869865 -> xyz=0.25 0.125 -0.0566 rpy=3.14159265359 0.0 0.50709869865
- joint hip_yaw_2: limit lower=-2.35619449 upper=0.78539816 effort=304 velocity=8.8 -> lower=-2.70526034 upper=1.13446401 effort=304 velocity=8.8; origin xyz=0.225 -0.125 0.11 rpy=3.14159265359 0.0 -0.50709869865 -> xyz=0.25 -0.125 -0.0566 rpy=3.14159265359 0.0 -0.50709869865
- joint hip_yaw_3: limit lower=-2.35619449 upper=0.78539816 effort=304 velocity=8.8 -> lower=-2.70526034 upper=1.13446401 effort=304 velocity=8.8; origin xyz=-0.225 0.125 0.11 rpy=3.14159265359 0.0 2.63449395494 -> xyz=-0.25 0.125 -0.0566 rpy=3.14159265359 0.0 2.63449395494
- joint hip_yaw_4: limit lower=-0.78539816 upper=2.35619449 effort=304 velocity=8.8 -> lower=-1.13446401 upper=2.70526034 effort=304 velocity=8.8; origin xyz=-0.225 -0.125 0.11 rpy=3.14159265359 0.0 3.64869135224 -> xyz=-0.25 -0.125 -0.0566 rpy=3.14159265359 0.0 3.64869135224
- joint imu_joint: origin xyz=-0.0704 0.0 -0.0416 -> xyz=0.0 0.0 0.0 rpy=0.0 0.0 0.0
- joint j_arm1_1: origin xyz=0.04576 0.169137 0.190626 rpy=0.0 0.0 -0.523602668986 -> xyz=0.04576 0.169137 0.116626 rpy=0.0 0.0 -0.523602668986
- joint j_arm1_8: type fixed -> revolute
- joint j_arm2_1: origin xyz=0.04576 -0.169137 0.190626 rpy=0.0 0.0 0.523602668986 -> xyz=0.04576 -0.169137 0.116626 rpy=0.0 0.0 0.523602668986
- joint j_arm2_8: type fixed -> revolute
- joint reference: origin xyz=0.0 0.0 0.759 -> xyz=0.0 0.0 0.9256
- joint torso_yaw: origin xyz=0.175 0.0 0.36 -> xyz=0.2 0.0 0.256

Commit message: version working on the robot computer
* change joint site position to motor site position
* imu state estimation
* gravity test - command velocities

File: locomotion_framework/xbot/robot_class_xbot/include/configs/urdf/centauro.urdf (robot description, URDF)
Before this commit: robot centauro, 44 links, 43 joints
Links:
- removed link pelvis_imu_link
- added link imu_link, mass 0.0
Joints:
- removed joint pelvis_imu_joint
- added joint imu_joint: type fixed, parent pelvis, child imu_link, origin xyz=0.0 0.0 0.0 rpy=0.0 0.0 0.0

Commit message: wheels with static stability

File: locomotion_framework/xbot/robot_class_xbot/include/configs/urdf/centauro.urdf (robot description, URDF)
Before this commit: robot centauro, 44 links, 43 joints
Links:
- link arm1_8: geometry collision mesh filename=package://centauro/centauro_urdf/meshes/convex_hull/link9.s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 scale=0.001 -0.001 -0.001; visual mesh filename=package://centauro/centauro_urdf/meshes/link9.stl scale=0.001 -0.001 -0.001
Joints:
- joint j_arm1_8: axis (none) -> 1 0 0
- joint j_arm2_8: axis (none) -> 1 0 0
- joint j_wheel_1: origin xyz=0.0 0.00085 0.235 rpy=1.57079632679 0.0 0.0 -> xyz=0.0 0.00085 0.237350 rpy=1.57079632679 0.0 3.14159265359
- joint j_wheel_2: origin xyz=0.0 0.00085 0.235 rpy=1.57079632679 0.0 0.0 -> xyz=0.0 0.00085 0.237350 rpy=1.57079632679 0.0 3.14159265359
- joint j_wheel_3: origin xyz=0.0 0.00085 0.235 rpy=1.57079632679 0.0 0.0 -> xyz=0.0 0.00085 0.237350 rpy=1.57079632679 0.0 3.14159265359
- joint j_wheel_4: origin xyz=0.0 0.00085 0.235 rpy=1.57079632679 0.0 0.0 -> xyz=0.0 0.00085 0.237350 rpy=1.57079632679 0.0 3.14159265359
- joint reference: origin xyz=0.0 0.0 0.9256 -> xyz=0.0 0.0 0.92795000

File: locomotion_framework/xbot/robot_class_xbot/include/configs/urdf/centauro_lower_body.urdf (robot description, URDF)
Before this commit: robot centauro, 27 links, 26 joints
Joints:
- joint j_wheel_1: origin xyz=0.0 0.00085 0.235 rpy=1.57079632679 0.0 0.0 -> xyz=0.0 0.00085 0.237350 rpy=1.57079632679 0.0 3.14159265359
- joint j_wheel_2: origin xyz=0.0 0.00085 0.235 rpy=1.57079632679 0.0 0.0 -> xyz=0.0 0.00085 0.237350 rpy=1.57079632679 0.0 3.14159265359
- joint j_wheel_3: origin xyz=0.0 0.00085 0.235 rpy=1.57079632679 0.0 0.0 -> xyz=0.0 0.00085 0.237350 rpy=1.57079632679 0.0 3.14159265359
- joint j_wheel_4: origin xyz=0.0 0.00085 0.235 rpy=1.57079632679 0.0 0.0 -> xyz=0.0 0.00085 0.237350 rpy=1.57079632679 0.0 3.14159265359
- joint reference: origin xyz=0.0 0.0 0.9256 -> xyz=0.0 0.0 0.92795000

Commit message: Define references, move tunning to config files

File: locomotion_framework/xbot/robot_class_xbot/include/configs/urdf/centauro.urdf (robot description, URDF)
Before this commit: robot centauro, 57 links, 56 joints
Links:
- removed link fl_foot_ft
- removed link foot_fl
- removed link foot_fr
- removed link foot_hl
- removed link foot_hr
- removed link fr_foot_ft
- removed link ft_arm1
- removed link ft_arm2
- removed link hl_foot_ft
- removed link hr_foot_ft
- removed link neck_1
- removed link neck_2
- removed link neck_3
Joints:
- removed joint j_fl_foot_ft
- removed joint j_foot_fl
- removed joint j_foot_fr
- removed joint j_foot_hl
- removed joint j_foot_hr
- removed joint j_fr_foot_ft
- removed joint j_ft_arm1
- removed joint j_ft_arm2
- removed joint j_hl_foot_ft
- removed joint j_hr_foot_ft
- removed joint neck_pitch
- removed joint neck_velodyne
- removed joint neck_yaw
- joint hip_pitch_1: origin xyz=0.0 0.0 0.059 rpy=1.57079632679 0.0 0.50709869865 -> xyz=0.0 0.0 0.0625 rpy=1.57079632679 0.0 0.46141612323
- joint hip_pitch_2: origin xyz=0.0 0.0 0.059 rpy=1.57079632679 0.0 2.63449395494 -> xyz=0.0 0.0 0.0625 rpy=1.57079632679 0.0 2.68017653036
- joint hip_pitch_3: origin xyz=0.0 0.0 0.059 rpy=1.57079632679 0.0 2.63449395494 -> xyz=0.0 0.0 0.0625 rpy=1.57079632679 0.0 2.68017653036
- joint hip_pitch_4: origin xyz=0.0 0.0 0.059 rpy=1.57079632679 0.0 0.50709869865 -> xyz=0.0 0.0 0.0625 rpy=1.57079632679 0.0 0.46141612323
- joint hip_yaw_1: origin xyz=0.25 0.125 -0.0566 rpy=3.14159265359 0.0 0.50709869865 -> xyz=0.25 0.125 -0.0566 rpy=3.14159265359 0.0 0.461416123228
- joint hip_yaw_2: origin xyz=0.25 -0.125 -0.0566 rpy=3.14159265359 0.0 -0.50709869865 -> xyz=0.25 -0.125 -0.0566 rpy=3.14159265359 0.0 -0.461416123228
- joint hip_yaw_3: origin xyz=-0.25 0.125 -0.0566 rpy=3.14159265359 0.0 2.63449395494 -> xyz=-0.25 0.125 -0.0566 rpy=3.14159265359 0.0 2.68017653036
- joint hip_yaw_4: origin xyz=-0.25 -0.125 -0.0566 rpy=3.14159265359 0.0 3.64869135224 -> xyz=-0.25 -0.125 -0.0566 rpy=3.14159265359 0.0 3.60300877682
- joint j_arm1_2: limit lower=-3.49 upper=-0.25 effort=147 velocity=5.7 -> lower=-3.49 upper=0 effort=147 velocity=5.7
- joint j_arm1_8: limit lower=0.0 upper=0 effort=0 velocity=0 -> (none)
- joint j_arm2_2: limit lower=0.25 upper=3.49 effort=147 velocity=5.7 -> lower=0 upper=3.49 effort=147 velocity=5.7
- joint j_arm2_8: limit lower=0.0 upper=0 effort=0 velocity=0 -> (none)
- joint j_wheel_1: limit lower=-1000000000000000 upper=1000000000000000 effort=35 velocity=20.0 -> effort=35 velocity=20.0; origin xyz=0.0 0.00085 0.235 rpy=1.57079632679 0.0 0.0 -> xyz=0.0 0.00085 0.23735 rpy=1.57079632679 0.0 3.14159265359
- joint j_wheel_2: limit lower=-1000000000000000 upper=1000000000000000 effort=35 velocity=20.0 -> effort=35 velocity=20.0; origin xyz=0.0 0.00085 0.235 rpy=1.57079632679 0.0 0.0 -> xyz=0.0 0.00085 0.23735 rpy=1.57079632679 0.0 3.14159265359
- joint j_wheel_3: limit lower=-1000000000000000 upper=1000000000000000 effort=35 velocity=20.0 -> effort=35 velocity=20.0; origin xyz=0.0 0.00085 0.235 rpy=1.57079632679 0.0 0.0 -> xyz=0.0 0.00085 0.23735 rpy=1.57079632679 0.0 3.14159265359
- joint j_wheel_4: limit lower=-1000000000000000 upper=1000000000000000 effort=35 velocity=20.0 -> effort=35 velocity=20.0; origin xyz=0.0 0.00085 0.235 rpy=1.57079632679 0.0 0.0 -> xyz=0.0 0.00085 0.23735 rpy=1.57079632679 0.0 3.14159265359
- joint reference: origin xyz=0.0 0.0 0.9256 -> xyz=0.0 0.0 0.93445

Commit message: updates from experiments

File: locomotion_framework/xbot/robot_class_xbot/include/configs/urdf/centauro.urdf (robot description, URDF)
Before this commit: robot centauro, 44 links, 43 joints
Joints:
- joint ankle_yaw_1: limit lower=-2.79252680 upper=2.79252680 effort=35 velocity=20.0 -> lower=-2.58 upper=2.58 effort=35 velocity=20.0
- joint ankle_yaw_2: limit lower=-2.79252680 upper=2.79252680 effort=35 velocity=20.0 -> lower=-2.58 upper=2.58 effort=35 velocity=20.0
- joint ankle_yaw_3: limit lower=-2.79252680 upper=2.79252680 effort=35 velocity=20.0 -> lower=-2.58 upper=2.58 effort=35 velocity=20.0
- joint ankle_yaw_4: limit lower=-2.79252680 upper=2.79252680 effort=35 velocity=20.0 -> lower=-2.58 upper=2.58 effort=35 velocity=20.0
- joint hip_yaw_1: limit lower=-1.13446401 upper=2.70526034 effort=304 velocity=8.8 -> lower=-0.975 upper=2.54 effort=304 velocity=8.8
- joint hip_yaw_2: limit lower=-2.70526034 upper=1.13446401 effort=304 velocity=8.8 -> lower=-2.54 upper=0.975 effort=304 velocity=8.8
- joint hip_yaw_3: limit lower=-2.70526034 upper=1.13446401 effort=304 velocity=8.8 -> lower=-2.54 upper=0.975 effort=304 velocity=8.8
- joint hip_yaw_4: limit lower=-1.13446401 upper=2.70526034 effort=304 velocity=8.8 -> lower=-0.975 upper=2.54 effort=304 velocity=8.8

Commit message: hand marge with RT changes

File: locomotion_framework/xbot/robot_class_xbot/include/configs/urdf/centauro.urdf (robot description, URDF)
Before this commit: robot centauro, 44 links, 43 joints
Links:
- removed link imu_link
- added link pelvis_imu_link, mass 0.0
- link arm1_8: geometry collision mesh filename=package://centauro/centauro_urdf/meshes/convex_hull/link9.s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 scale=0.001 -0.001 -0.001
Joints:
- removed joint imu_joint
- added joint pelvis_imu_joint: type fixed, parent pelvis, child pelvis_imu_link, origin xyz=0.0 0.0 0.0 rpy=0.0 0.0 0.0
- joint hip_pitch_1: origin xyz=0.0 0.0 0.0625 rpy=1.57079632679 0.0 0.46141612323 -> xyz=0.0 0.0 0.059 rpy=1.57079632679 0.0 0.50709869865
- joint hip_pitch_2: origin xyz=0.0 0.0 0.0625 rpy=1.57079632679 0.0 2.68017653036 -> xyz=0.0 0.0 0.059 rpy=1.57079632679 0.0 2.63449395494
- joint hip_pitch_3: origin xyz=0.0 0.0 0.0625 rpy=1.57079632679 0.0 2.68017653036 -> xyz=0.0 0.0 0.059 rpy=1.57079632679 0.0 2.63449395494
- joint hip_pitch_4: origin xyz=0.0 0.0 0.0625 rpy=1.57079632679 0.0 0.46141612323 -> xyz=0.0 0.0 0.059 rpy=1.57079632679 0.0 0.50709869865
- joint hip_yaw_1: origin xyz=0.25 0.125 -0.0566 rpy=3.14159265359 0.0 0.461416123228 -> xyz=0.25 0.125 -0.0566 rpy=3.14159265359 0.0 0.50709869865
- joint hip_yaw_2: origin xyz=0.25 -0.125 -0.0566 rpy=3.14159265359 0.0 -0.461416123228 -> xyz=0.25 -0.125 -0.0566 rpy=3.14159265359 0.0 -0.50709869865
- joint hip_yaw_3: origin xyz=-0.25 0.125 -0.0566 rpy=3.14159265359 0.0 2.68017653036 -> xyz=-0.25 0.125 -0.0566 rpy=3.14159265359 0.0 2.63449395494
- joint hip_yaw_4: origin xyz=-0.25 -0.125 -0.0566 rpy=3.14159265359 0.0 3.60300877682 -> xyz=-0.25 -0.125 -0.0566 rpy=3.14159265359 0.0 3.64869135224
- joint j_arm1_8: axis 1 0 0 -> (none)
- joint j_arm2_8: axis 1 0 0 -> (none)
- joint j_wheel_1: origin xyz=0.0 0.00085 0.23735 rpy=1.57079632679 0.0 3.14159265359 -> xyz=0.0 0.00085 0.235 rpy=1.57079632679 0.0 0.0
- joint j_wheel_2: origin xyz=0.0 0.00085 0.23735 rpy=1.57079632679 0.0 3.14159265359 -> xyz=0.0 0.00085 0.235 rpy=1.57079632679 0.0 0.0
- joint j_wheel_3: origin xyz=0.0 0.00085 0.23735 rpy=1.57079632679 0.0 3.14159265359 -> xyz=0.0 0.00085 0.235 rpy=1.57079632679 0.0 0.0
- joint j_wheel_4: origin xyz=0.0 0.00085 0.23735 rpy=1.57079632679 0.0 3.14159265359 -> xyz=0.0 0.00085 0.235 rpy=1.57079632679 0.0 0.0
- joint reference: origin xyz=0.0 0.0 0.93445 -> xyz=0.0 0.0 0.9256
