Commit message: working experiments

File: configs/xbot/centauro.urdf (robot description, URDF)
Before this commit: robot centauro, 44 links, 43 joints
Links:
- added link HeriDown_link, mass 2.0
- added link HeriEnd_link, mass 2.0
- added link HeriUp_link, mass 2.0
- added link foot_fl, mass 0; visual box size=0.01 0.01 0.01
- added link foot_fr, mass 0; visual box size=0.01 0.01 0.01
- added link foot_hl, mass 0; visual box size=0.01 0.01 0.01
- added link foot_hr, mass 0; visual box size=0.01 0.01 0.01
- added link ft_arm1, mass 0.15; collision mesh filename=package://centauro/centauro_urdf/meshes/link9.stl scale=0.001 0.001 -0.001; visual mesh filename=package://centauro/centauro_urdf/meshes/simplified/link9.stl scale=0.001 0.001 -0.001
- added link ft_arm2, mass 0.15; collision mesh filename=package://centauro/centauro_urdf/meshes/link9.stl scale=0.001 0.001 -0.001; visual mesh filename=package://centauro/centauro_urdf/meshes/simplified/link9.stl scale=0.001 0.001 -0.001
- added link neck_1, mass 0.33878686; collision mesh filename=package://centauro/centauro_urdf/meshes/convex_hull/neck_ya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 scale=0.001 0.001 0.001; visual mesh filename=package://centauro/centauro_urdf/meshes/simplified/neck_yaw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 scale=0.001 0.001 0.001
- added link neck_2, mass 0.78526942; collision mesh filename=package://centauro/centauro_urdf/meshes/convex_hull/neck_pi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 scale=0.001 0.001 0.001; visual mesh filename=package://centauro/centauro_urdf/meshes/simplified/neck_pit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 scale=0.001 0.001 0.001
- added link neck_3, mass 0.78526942; collision mesh filename=package://centauro/centauro_urdf/meshes/convex_hull/velodyn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 scale=0.001 0.001 0.001; visual mesh filename=package://centauro/centauro_urdf/meshes/simplified/velodyne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 scale=0.001 0.001 0.001
- link ankle1_1: geometry collision mesh filename=package://centauro/centauro_urdf/meshes/convex_hull/ankle-p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 scale=0.001 0.001 0.001; visual mesh filename=package://centauro/centauro_urdf/meshes/simplified/ankle-pi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 scale=0.001 0.001 0.001
- link ankle1_2: geometry collision mesh filename=package://centauro/centauro_urdf/meshes/convex_hull/ankle-p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 scale=0.001 0.001 0.001; visual mesh filename=package://centauro/centauro_urdf/meshes/simplified/ankle-pi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 scale=0.001 0.001 0.001
- link ankle1_3: geometry collision mesh filename=package://centauro/centauro_urdf/meshes/convex_hull/ankle-p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 scale=0.001 0.001 0.001; visual mesh filename=package://centauro/centauro_urdf/meshes/simplified/ankle-pi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 scale=0.001 0.001 0.001
- link ankle1_4: geometry collision mesh filename=package://centauro/centauro_urdf/meshes/convex_hull/ankle-p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 scale=0.001 0.001 0.001; visual mesh filename=package://centauro/centauro_urdf/meshes/simplified/ankle-pi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 scale=0.001 0.001 0.001
- link ankle2_1: geometry collision mesh filename=package://centauro/centauro_urdf/meshes/convex_hull/ankle-y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 scale=0.001 0.001 0.001; visual mesh filename=package://centauro/centauro_urdf/meshes/simplified/ankle-ya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 scale=0.001 0.001 0.001
- link ankle2_2: geometry collision mesh filename=package://centauro/centauro_urdf/meshes/convex_hull/ankle-y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 scale=0.001 0.001 0.001; visual mesh filename=package://centauro/centauro_urdf/meshes/simplified/ankle-ya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 scale=0.001 0.001 0.001
- link ankle2_3: geometry collision mesh filename=package://centauro/centauro_urdf/meshes/convex_hull/ankle-y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 scale=0.001 0.001 0.001; visual mesh filename=package://centauro/centauro_urdf/meshes/simplified/ankle-ya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 scale=0.001 0.001 0.001
- link ankle2_4: geometry collision mesh filename=package://centauro/centauro_urdf/meshes/convex_hull/ankle-y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 scale=0.001 0.001 0.001; visual mesh filename=package://centauro/centauro_urdf/meshes/simplified/ankle-ya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 scale=0.001 0.001 0.001
- link arm1_1: geometry collision mesh filename=package://centauro/centauro_urdf/meshes/convex_hull/link2.s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 scale=0.001 -0.001 0.001; visual mesh filename=package://centauro/centauro_urdf/meshes/simplified/link2.stl scale=0.001 -0.001 0.001
- link arm1_2: geometry collision mesh filename=package://centauro/centauro_urdf/meshes/convex_hull/link3.s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 scale=0.001 -0.001 0.001; visual mesh filename=package://centauro/centauro_urdf/meshes/simplified/link3.stl scale=0.001 -0.001 0.001
- link arm1_3: geometry collision mesh filename=package://centauro/centauro_urdf/meshes/convex_hull/link4.s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 scale=0.001 -0.001 0.001; visual mesh filename=package://centauro/centauro_urdf/meshes/simplified/link4.stl scale=0.001 -0.001 0.001
- link arm1_4: geometry collision mesh filename=package://centauro/centauro_urdf/meshes/convex_hull/link5.s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 scale=0.001 -0.001 0.001; visual mesh filename=package://centauro/centauro_urdf/meshes/simplified/link5.stl scale=0.001 -0.001 0.001
- link arm1_5: geometry collision mesh filename=package://centauro/centauro_urdf/meshes/convex_hull/link6.s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 scale=0.001 -0.001 0.001; visual mesh filename=package://centauro/centauro_urdf/meshes/simplified/link6.stl scale=0.001 -0.001 0.001
- link arm1_6: geometry collision mesh filename=package://centauro/centauro_urdf/meshes/convex_hull/link7.s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 scale=0.001 -0.001 0.001; visual mesh filename=package://centauro/centauro_urdf/meshes/simplified/link7.stl scale=0.001 -0.001 0.001
- link arm1_7: geometry collision mesh filename=package://centauro/centauro_urdf/meshes/convex_hull/link8.s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 scale=0.001 -0.001 0.001; visual mesh filename=package://centauro/centauro_urdf/meshes/simplified/link8.stl scale=0.001 -0.001 0.001
- link arm1_8: geometry collision mesh filename=package://centauro/centauro_urdf/meshes/convex_hull/link9.s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 scale=0.001 -0.001 -0.001; visual mesh filename=package://centauro/centauro_urdf/meshes/simplified/link9.stl scale=0.001 -0.001 -0.001
- link arm2_1: geometry collision mesh filename=package://centauro/centauro_urdf/meshes/convex_hull/link2.s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 scale=0.001 0.001 0.001; visual mesh filename=package://centauro/centauro_urdf/meshes/simplified/link2.stl scale=0.001 0.001 0.001
- link arm2_2: geometry collision mesh filename=package://centauro/centauro_urdf/meshes/convex_hull/link3.s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 scale=0.001 0.001 0.001; visual mesh filename=package://centauro/centauro_urdf/meshes/simplified/link3.stl scale=0.001 0.001 0.001
- link arm2_3: geometry collision mesh filename=package://centauro/centauro_urdf/meshes/convex_hull/link4.s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 scale=0.001 0.001 0.001; visual mesh filename=package://centauro/centauro_urdf/meshes/simplified/link4.stl scale=0.001 0.001 0.001
- link arm2_4: geometry collision mesh filename=package://centauro/centauro_urdf/meshes/convex_hull/link5.s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 scale=0.001 0.001 0.001; visual mesh filename=package://centauro/centauro_urdf/meshes/simplified/link5.stl scale=0.001 0.001 0.001
- link arm2_5: geometry collision mesh filename=package://centauro/centauro_urdf/meshes/convex_hull/link6.s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 scale=0.001 0.001 0.001; visual mesh filename=package://centauro/centauro_urdf/meshes/simplified/link6.stl scale=0.001 0.001 0.001
- link arm2_6: geometry collision mesh filename=package://centauro/centauro_urdf/meshes/convex_hull/link7.s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 scale=0.001 0.001 0.001; visual mesh filename=package://centauro/centauro_urdf/meshes/simplified/link7.stl scale=0.001 0.001 0.001
- link arm2_7: geometry collision mesh filename=package://centauro/centauro_urdf/meshes/convex_hull/link8.s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 scale=0.001 0.001 0.001; visual mesh filename=package://centauro/centauro_urdf/meshes/simplified/link8.stl scale=0.001 0.001 0.001
- link arm2_8: geometry collision mesh filename=package://centauro/centauro_urdf/meshes/convex_hull/link9.s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 scale=0.001 0.001 -0.001; visual mesh filename=package://centauro/centauro_urdf/meshes/simplified/link9.stl scale=0.001 0.001 -0.001
- link hip1_1: geometry collision mesh filename=package://centauro/centauro_urdf/meshes/convex_hull/hip-yaw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 scale=0.001 0.001 0.001; visual mesh filename=package://centauro/centauro_urdf/meshes/simplified/hip-yaw.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 scale=0.001 0.001 0.001
- link hip1_2: geometry collision mesh filename=package://centauro/centauro_urdf/meshes/convex_hull/hip-yaw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 scale=0.001 0.001 0.001; visual mesh filename=package://centauro/centauro_urdf/meshes/simplified/hip-yaw.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 scale=0.001 0.001 0.001
- link hip1_3: geometry collision mesh filename=package://centauro/centauro_urdf/meshes/convex_hull/hip-yaw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 scale=0.001 0.001 0.001; visual mesh filename=package://centauro/centauro_urdf/meshes/simplified/hip-yaw.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 scale=0.001 0.001 0.001
- link hip1_4: geometry collision mesh filename=package://centauro/centauro_urdf/meshes/convex_hull/hip-yaw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 scale=0.001 0.001 0.001; visual mesh filename=package://centauro/centauro_urdf/meshes/simplified/hip-yaw.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 scale=0.001 0.001 0.001
- link hip2_1: geometry collision mesh filename=package://centauro/centauro_urdf/meshes/convex_hull/hip-pit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 scale=0.001 0.001 0.001; visual mesh filename=package://centauro/centauro_urdf/meshes/simplified/hip-pitc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 scale=0.001 0.001 0.001
- link hip2_2: geometry collision mesh filename=package://centauro/centauro_urdf/meshes/convex_hull/hip-pit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 scale=0.001 0.001 0.001; visual mesh filename=package://centauro/centauro_urdf/meshes/simplified/hip-pitc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 scale=0.001 0.001 0.001
- link hip2_3: geometry collision mesh filename=package://centauro/centauro_urdf/meshes/convex_hull/hip-pit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 scale=0.001 0.001 0.001; visual mesh filename=package://centauro/centauro_urdf/meshes/simplified/hip-pitc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 scale=0.001 0.001 0.001
- link hip2_4: geometry collision mesh filename=package://centauro/centauro_urdf/meshes/convex_hull/hip-pit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 scale=0.001 0.001 0.001; visual mesh filename=package://centauro/centauro_urdf/meshes/simplified/hip-pitc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 scale=0.001 0.001 0.001
- link knee_1: geometry collision mesh filename=package://centauro/centauro_urdf/meshes/convex_hull/knee.stl scale=0.001 0.001 0.001; visual mesh filename=package://centauro/centauro_urdf/meshes/simplified/knee.stl scale=0.001 0.001 0.001
- link knee_2: geometry collision mesh filename=package://centauro/centauro_urdf/meshes/convex_hull/knee.stl scale=0.001 0.001 0.001; visual mesh filename=package://centauro/centauro_urdf/meshes/simplified/knee.stl scale=0.001 0.001 0.001
- link knee_3: geometry collision mesh filename=package://centauro/centauro_urdf/meshes/convex_hull/knee.stl scale=0.001 0.001 0.001; visual mesh filename=package://centauro/centauro_urdf/meshes/simplified/knee.stl scale=0.001 0.001 0.001
- link knee_4: geometry collision mesh filename=package://centauro/centauro_urdf/meshes/convex_hull/knee.stl scale=0.001 0.001 0.001; visual mesh filename=package://centauro/centauro_urdf/meshes/simplified/knee.stl scale=0.001 0.001 0.001
- link pelvis: geometry collision mesh filename=package://centauro/centauro_urdf/meshes/convex_hull/pelvis.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 scale=0.001 0.001 0.001; visual mesh filename=package://centauro/centauro_urdf/meshes/simplified/pelvis.s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 scale=0.001 0.001 0.001
- link torso_2: geometry collision mesh filename=package://centauro/centauro_urdf/meshes/convex_hull/link1.s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 scale=0.001 0.001 0.001; visual mesh filename=package://centauro/centauro_urdf/meshes/simplified/link1.stl scale=0.001 0.001 0.001
- link wheel_1: geometry collision mesh filename=package://centauro/centauro_urdf/meshes/convex_hull/wheel.s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 scale=0.001 0.001 0.001; visual mesh filename=package://centauro/centauro_urdf/meshes/simplified/wheel.stl scale=0.001 0.001 0.001
- link wheel_2: geometry collision mesh filename=package://centauro/centauro_urdf/meshes/convex_hull/wheel.s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 scale=0.001 0.001 0.001; visual mesh filename=package://centauro/centauro_urdf/meshes/simplified/wheel.stl scale=0.001 0.001 0.001
- link wheel_3: geometry collision mesh filename=package://centauro/centauro_urdf/meshes/convex_hull/wheel.s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 scale=0.001 0.001 0.001; visual mesh filename=package://centauro/centauro_urdf/meshes/simplified/wheel.stl scale=0.001 0.001 0.001
- link wheel_4: geometry collision mesh filename=package://centauro/centauro_urdf/meshes/convex_hull/wheel.s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 scale=0.001 0.001 0.001; visual mesh filename=package://centauro/centauro_urdf/meshes/simplified/wheel.stl scale=0.001 0.001 0.001
Joints:
- added joint 110: type fixed, parent HeriDown_link, child HeriUp_link, origin xyz=0 0 0.11 rpy=0 0 0, axis 0 0 1
- added joint 111: type fixed, parent HeriUp_link, child HeriEnd_link, origin xyz=0 0 0.2005 rpy=0 0 0, axis 0 -1 0
- added joint HeriBase: type fixed, parent arm1_8, child HeriDown_link, origin xyz=0 0 0 rpy=0 0 0
- added joint j_foot_fl: type fixed, parent ankle2_1, child foot_fl, origin xyz=0.0 0.0 0.30 rpy=3.1415 0.0 3.1415
- added joint j_foot_fr: type fixed, parent ankle2_2, child foot_fr, origin xyz=0.0 0.0 0.30 rpy=3.1415 0.0 0.0
- added joint j_foot_hl: type fixed, parent ankle2_3, child foot_hl, origin xyz=0.0 0.0 0.30 rpy=3.1415 0.0 3.1415
- added joint j_foot_hr: type fixed, parent ankle2_4, child foot_hr, origin xyz=0.0 0.0 0.30 rpy=3.1415 0.0 0.0
- added joint j_ft_arm1: type fixed, parent arm1_7, child ft_arm1, origin xyz=0.0 0.0 -0.0405 rpy=0.0 3.14159265359 -3.14159265359, axis 1 0 0, limit lower=0.0 upper=0 effort=0 velocity=0
- added joint j_ft_arm2: type fixed, parent arm2_7, child ft_arm2, origin xyz=0.0 0.0 -0.0405 rpy=0.0 3.14159265359 -3.14159265359, axis 1 0 0, limit lower=0.0 upper=0 effort=0 velocity=0
- added joint neck_pitch: type revolute, parent neck_1, child neck_2, origin xyz=0.054 0.0596 -0.0124975, axis 0 1 0, limit lower=-0.34906585 upper=0.78539816 effort=35 velocity=5.7
- added joint neck_velodyne: type continuous, parent torso_2, child neck_3, origin xyz=0.055 0.0 0.473262, axis 0 0 1, limit lower=-1000000000000000 upper=1000000000000000 effort=35 velocity=5.7
- added joint neck_yaw: type revolute, parent torso_2, child neck_1, origin xyz=0.0 0.0 0.2795, axis 0 0 1, limit lower=-0.78539816 upper=0.78539816 effort=35 velocity=5.7
- joint hip_pitch_1: origin xyz=0.0 0.0 0.0625 rpy=1.57079632679 0.0 0.46141612323 -> xyz=0.0 0.0 0.059 rpy=1.57079632679 0.0 0.50709869865
- joint hip_pitch_2: origin xyz=0.0 0.0 0.0625 rpy=1.57079632679 0.0 2.68017653036 -> xyz=0.0 0.0 0.059 rpy=1.57079632679 0.0 2.63449395494
- joint hip_pitch_3: origin xyz=0.0 0.0 0.0625 rpy=1.57079632679 0.0 2.68017653036 -> xyz=0.0 0.0 0.059 rpy=1.57079632679 0.0 2.63449395494
- joint hip_pitch_4: origin xyz=0.0 0.0 0.0625 rpy=1.57079632679 0.0 0.46141612323 -> xyz=0.0 0.0 0.059 rpy=1.57079632679 0.0 0.50709869865
- joint hip_yaw_1: origin xyz=0.25 0.125 -0.0566 rpy=3.14159265359 0.0 0.461416123228 -> xyz=0.25 0.125 -0.0566 rpy=3.14159265359 0.0 0.50709869865
- joint hip_yaw_2: origin xyz=0.25 -0.125 -0.0566 rpy=3.14159265359 0.0 -0.461416123228 -> xyz=0.25 -0.125 -0.0566 rpy=3.14159265359 0.0 -0.50709869865
- joint hip_yaw_3: origin xyz=-0.25 0.125 -0.0566 rpy=3.14159265359 0.0 2.68017653036 -> xyz=-0.25 0.125 -0.0566 rpy=3.14159265359 0.0 2.63449395494
- joint hip_yaw_4: origin xyz=-0.25 -0.125 -0.0566 rpy=3.14159265359 0.0 3.60300877682 -> xyz=-0.25 -0.125 -0.0566 rpy=3.14159265359 0.0 3.64869135224
- joint j_arm1_1: axis 0 0.984807753012 0.173648177667 -> (none); limit lower=-3.403 upper=1.658 effort=147 velocity=5.7 -> (none)
- joint j_arm1_2: axis -1 0 0 -> (none); limit lower=-3.49 upper=0 effort=147 velocity=5.7 -> (none)
- joint j_arm1_3: axis 0 0 -1 -> (none); limit lower=-2.618 upper=2.618 effort=147 velocity=8.2 -> (none)
- joint j_arm1_4: axis 0 1 0 -> (none); limit lower=-2.530 upper=0.349 effort=147 velocity=8.2 -> (none)
- joint j_arm1_5: axis 0 0 -1 -> (none); limit lower=-2.618 upper=2.618 effort=55 velocity=11.6 -> (none)
- joint j_arm1_6: axis 0 1 0 -> (none); limit lower=-1.570 upper=1.570 effort=55 velocity=11.6 -> (none)
- joint j_arm1_7: axis 0 0 -1 -> (none); limit lower=-2.618 upper=2.618 effort=27 velocity=20.3 -> (none)
- joint j_arm1_8: limit (none) -> lower=0.0 upper=0 effort=0 velocity=0
- joint j_arm2_2: limit lower=0 upper=3.49 effort=147 velocity=5.7 -> lower=0.25 upper=3.49 effort=147 velocity=5.7
- joint j_arm2_8: limit (none) -> lower=0.0 upper=0 effort=0 velocity=0
- joint j_wheel_1: axis 0 0 1 -> 0 0 -1; limit effort=35 velocity=20.0 -> lower=-1000000000000000 upper=1000000000000000 effort=35 velocity=20.0; origin xyz=0.0 0.00085 0.23735 rpy=1.57079632679 0.0 3.14159265359 -> xyz=0.0 0.00085 0.235 rpy=1.57079632679 0.0 0.0
- joint j_wheel_2: axis 0 0 1 -> 0 0 -1; limit effort=35 velocity=20.0 -> lower=-1000000000000000 upper=1000000000000000 effort=35 velocity=20.0; origin xyz=0.0 0.00085 0.23735 rpy=1.57079632679 0.0 3.14159265359 -> xyz=0.0 0.00085 0.235 rpy=1.57079632679 0.0 0.0
- joint j_wheel_3: axis 0 0 1 -> 0 0 -1; limit effort=35 velocity=20.0 -> lower=-1000000000000000 upper=1000000000000000 effort=35 velocity=20.0; origin xyz=0.0 0.00085 0.23735 rpy=1.57079632679 0.0 3.14159265359 -> xyz=0.0 0.00085 0.235 rpy=1.57079632679 0.0 0.0
- joint j_wheel_4: axis 0 0 1 -> 0 0 -1; limit effort=35 velocity=20.0 -> lower=-1000000000000000 upper=1000000000000000 effort=35 velocity=20.0; origin xyz=0.0 0.00085 0.23735 rpy=1.57079632679 0.0 3.14159265359 -> xyz=0.0 0.00085 0.235 rpy=1.57079632679 0.0 0.0
- joint reference: origin xyz=0.0 0.0 0.93445 -> xyz=0.0 0.0 0.9256
