Commit message: Integrate shared control with xbot core

File: configs/mwoibn/urdf/centauro.urdf (robot description, URDF)
Before this commit: robot centauro, 53 links, 52 joints
Links:
- added link ft_arm1, mass 0.37827821; collision mesh filename=package://centauro/centauro_urdf/meshes/convex_hull/link9.s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 scale=0.001 -0.001 0.001; visual mesh filename=package://centauro/centauro_urdf/meshes/simplified/Wrist.STL scale=0.001 -0.001 0.001
- added link ft_arm2, mass 0.37827821; collision mesh filename=package://centauro/centauro_urdf/meshes/convex_hull/link9.s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 scale=0.001 0.001 0.001; visual mesh filename=package://centauro/centauro_urdf/meshes/simplified/Wrist.STL scale=0.001 0.001 0.001
- added link kinect2_rgb_frame
- added link velodyne_calib
- link arm1_1: mass 1.5583338 -> 1.9628675; geometry collision mesh filename=package://centauro/centauro_urdf/meshes/convex_hull/link2.s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 scale=0.001 -0.001 0.001; visual mesh filename=package://centauro/centauro_urdf/meshes/simplified/Shoulder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 scale=0.001 -0.001 0.001
- link arm1_2: mass 1.515061 -> 1.8595811; geometry collision mesh filename=package://centauro/centauro_urdf/meshes/convex_hull/link3.s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 scale=0.001 -0.001 0.001; visual mesh filename=package://centauro/centauro_urdf/meshes/simplified/Shoulder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 scale=0.001 -0.001 0.001
- link arm1_3: mass 1.5088101 -> 1.6678109; geometry collision mesh filename=package://centauro/centauro_urdf/meshes/convex_hull/link4.s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 scale=0.001 -0.001 0.001; visual mesh filename=package://centauro/centauro_urdf/meshes/simplified/Shoulder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 scale=0.001 -0.001 0.001
- link arm1_4: mass 0.96297329 -> 1.3157289; geometry collision mesh filename=package://centauro/centauro_urdf/meshes/convex_hull/link5.s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 scale=0.001 -0.001 0.001; visual mesh filename=package://centauro/centauro_urdf/meshes/simplified/Elbow.STL scale=0.001 -0.001 0.001
- link arm1_5: mass 1.4703698 -> 1.4908547; geometry collision mesh filename=package://centauro/centauro_urdf/meshes/convex_hull/link6.s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 scale=0.001 -0.001 0.001; visual mesh filename=package://centauro/centauro_urdf/meshes/simplified/Forearm.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 scale=0.001 -0.001 0.001
- link arm1_6: mass 0.94693868 -> 1.1263612; geometry collision mesh filename=package://centauro/centauro_urdf/meshes/convex_hull/link7.s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 scale=0.001 -0.001 0.001; visual mesh filename=package://centauro/centauro_urdf/meshes/simplified/ForearmP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 scale=0.001 -0.001 0.001
- link arm1_7: mass 0.55981036 -> 0.27966428; geometry collision mesh filename=package://centauro/centauro_urdf/meshes/convex_hull/link8.s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 scale=0.001 -0.001 0.001; visual mesh filename=package://centauro/centauro_urdf/meshes/simplified/ForearmY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 scale=0.001 -0.001 0.001
- link arm1_8: mass 0.15 -> 1.8366865; geometry collision mesh filename=package://centauro/centauro_urdf/meshes/convex_hull/heri.stl scale=0.001 -0.001 -0.001; visual mesh filename=package://centauro/centauro_urdf/meshes/simplified/heri.stl scale=0.001 -0.001 -0.001
- link arm2_1: mass 1.5583338 -> 1.9628675; geometry collision mesh filename=package://centauro/centauro_urdf/meshes/convex_hull/link2.s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 scale=0.001 0.001 0.001; visual mesh filename=package://centauro/centauro_urdf/meshes/simplified/Shoulder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 scale=0.001 0.001 0.001
- link arm2_2: mass 1.515061 -> 1.8595811; geometry collision mesh filename=package://centauro/centauro_urdf/meshes/convex_hull/link3.s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 scale=0.001 0.001 0.001; visual mesh filename=package://centauro/centauro_urdf/meshes/simplified/Shoulder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 scale=0.001 0.001 0.001
- link arm2_3: mass 1.5088101 -> 1.6678109; geometry collision mesh filename=package://centauro/centauro_urdf/meshes/convex_hull/link4.s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 scale=0.001 0.001 0.001; visual mesh filename=package://centauro/centauro_urdf/meshes/simplified/Shoulder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 scale=0.001 0.001 0.001
- link arm2_4: mass 0.96297329 -> 1.3157289; geometry collision mesh filename=package://centauro/centauro_urdf/meshes/convex_hull/link5.s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 scale=0.001 0.001 0.001; visual mesh filename=package://centauro/centauro_urdf/meshes/simplified/Elbow.STL scale=0.001 0.001 0.001
- link arm2_5: mass 1.4703698 -> 1.4908547; geometry collision mesh filename=package://centauro/centauro_urdf/meshes/convex_hull/link6.s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 scale=0.001 0.001 0.001; visual mesh filename=package://centauro/centauro_urdf/meshes/simplified/Forearm.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 scale=0.001 0.001 0.001
- link arm2_6: mass 0.94693868 -> 1.1263612; geometry collision mesh filename=package://centauro/centauro_urdf/meshes/convex_hull/link7.s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 scale=0.001 0.001 0.001; visual mesh filename=package://centauro/centauro_urdf/meshes/simplified/ForearmP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 scale=0.001 0.001 0.001
- link arm2_7: mass 0.55981036 -> 0.27966428; geometry collision mesh filename=package://centauro/centauro_urdf/meshes/convex_hull/link8.s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 scale=0.001 0.001 0.001; visual mesh filename=package://centauro/centauro_urdf/meshes/simplified/ForearmY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 scale=0.001 0.001 0.001
- link neck_3: geometry collision mesh filename=package://centauro/centauro_urdf/meshes/convex_hull/velodyn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 scale=0.001 0.001 0.001; visual mesh filename=package://centauro/centauro_urdf/meshes/simplified/mesh_lid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 scale=0.001 0.001 0.001
- link pelvis: mass 24.190945 -> 16.097574
- link torso_2: mass 6.1886404 -> 11.492689
Joints:
- added joint j_ft_1: type fixed, parent arm1_7, child ft_arm1, origin xyz=0.0 0.0 -0.0 rpy=0.0 0.0 0.0, axis 0 0 1, limit lower=0.0 upper=0.0 effort=0 velocity=0
- added joint j_ft_2: type fixed, parent arm2_7, child ft_arm2, origin xyz=0.0 0.0 -0.0 rpy=0.0 0.0 0.0, axis 0 0 1, limit lower=0.0 upper=0.0 effort=0 velocity=0
- added joint j_kinect2_rgb_frame: type fixed, parent kinect, child kinect2_rgb_frame, origin xyz=0.050 -0.110 -0.035
- added joint velodyne_calib: type fixed, parent neck_3, child velodyne_calib, origin xyz=-0.175768 0 -0.034219 rpy=-1.57772 0.0128311 1.57073
- joint hip_yaw_1: limit lower=-0.9432 upper=2.5138 effort=304 velocity=8.8 -> lower=-2.03 upper=1.2 effort=304 velocity=8.8
- joint hip_yaw_2: limit lower=-2.511 upper=0.943 effort=304 velocity=8.8 -> lower=-1.2 upper=2.03 effort=304 velocity=8.8
- joint hip_yaw_3: limit lower=-2.51 upper=0.943 effort=304 velocity=8.8 -> lower=-1.2 upper=2.03 effort=304 velocity=8.8
- joint hip_yaw_4: limit lower=-0.9412 upper=2.5138 effort=304 velocity=8.8 -> lower=-2.03 upper=1.2 effort=304 velocity=8.8
- joint imu_joint: origin xyz=0.0 0.0 0.0 rpy=0.0 0.0 0.0 -> xyz=0.248316 0.0 0.015 rpy=0.0 0.0 0.0
- joint j_arm1_1: axis 0 0.984807753012 0.173648177667 -> 0 1 0; limit lower=-3.348 upper=1.578 effort=147 velocity=5.7 -> lower=-3.312 upper=1.615 effort=147.0 velocity=3.86; origin xyz=0.04576 0.169137 0.116626 rpy=0.0 0.0 -0.523602668986 -> xyz=0.0457475 0.169137 0.116626 rpy=0.174533 0.0 -0.5235988
- joint j_arm1_2: axis -1 0 0 -> 1 0 0; limit lower=-3.42 upper=-0.056 effort=147 velocity=5.7 -> lower=0.02 upper=3.431 effort=147.0 velocity=3.86; origin xyz=-0.09115 0.06106 0.010766 -> xyz=-0.09015 0.062 0.0 rpy=-0.1745327 0.0 0.0
- joint j_arm1_3: axis 0 0 -1 -> 0 0 1; limit lower=-2.5556 upper=2.5424 effort=147 velocity=8.2 -> lower=-2.552 upper=2.566 effort=147.0 velocity=6.06; origin xyz=0.09115 0.0 -0.21915 -> xyz=0.09015 0.0 -0.21815
- joint j_arm1_4: limit lower=-2.4636 upper=0.2804 effort=147 velocity=8.2 -> lower=-2.465 upper=0.28 effort=147.0 velocity=6.06; origin xyz=0.04 0.05615 -0.074 -> xyz=0.045 0.05515 -0.074
- joint j_arm1_5: axis 0 0 -1 -> 0 0 1; limit lower=-2.5406 upper=2.5534 effort=55 velocity=11.6 -> lower=-2.569 upper=2.562 effort=55.0 velocity=11.72; origin xyz=-0.015 -0.05615 -0.061 -> xyz=-0.015 -0.05515 -0.095
- joint j_arm1_6: limit lower=-1.5096 upper=1.5044 effort=55 velocity=11.6 -> lower=-1.529 upper=1.509 effort=55.0 velocity=11.72; origin xyz=0.0 0.049 -0.18 -> xyz=0.0 0.049 -0.156
- joint j_arm1_7: axis 0 0 -1 -> 0 0 1; limit lower=-2.5376 upper=2.5554 effort=27 velocity=20.3 -> lower=-2.565 upper=2.569 effort=28.32 velocity=20.35; origin xyz=0.0 -0.049 -0.169 -> xyz=0.0 -0.049 -0.174
- joint j_arm1_8: origin xyz=0.0 0.0 -0.0405 rpy=0.0 3.14159265359 -1.5707963268 -> xyz=0.0 0.0 -0.0415 rpy=0.0 3.14159265359 3.14159265359; parent arm1_7 -> ft_arm1
- joint j_arm2_1: axis 0 -0.984807753012 0.173648177667 -> 0 1 0; limit lower=-1.6102 upper=3.3138 effort=147 velocity=5.7 -> lower=-3.3458 upper=1.6012 effort=147.0 velocity=3.86; origin xyz=0.04576 -0.169137 0.116626 rpy=0.0 0.0 0.523602668986 -> xyz=0.0457475 -0.169137 0.116626 rpy=0.174533 0.0 0.5235988
- joint j_arm2_2: axis -1 0 0 -> 1 0 0; limit lower=0.0578 upper=3.4288 effort=147 velocity=5.7 -> lower=-3.4258 upper=-0.0138 effort=147.0 velocity=3.86; origin xyz=-0.09115 -0.06106 0.010766 -> xyz=-0.09015 -0.062 0.0 rpy=-0.1745327 0.0 0.0
- joint j_arm2_3: axis 0 0 -1 -> 0 0 1; limit lower=-2.5426 upper=2.5524 effort=147 velocity=8.2 -> lower=-2.5614 upper=2.5606 effort=147.0 velocity=6.06; origin xyz=0.09115 0.0 -0.21915 -> xyz=0.09015 0.0 -0.21815
- joint j_arm2_4: axis 0 -1 0 -> 0 1 0; limit lower=-0.2796 upper=2.4564 effort=147 velocity=8.2 -> lower=-2.4794 upper=0.2886 effort=147.0 velocity=6.06; origin xyz=0.04 -0.05615 -0.074 -> xyz=0.045 -0.05515 -0.074
- joint j_arm2_5: axis 0 0 -1 -> 0 0 1; limit lower=-2.5626 upper=2.5464 effort=55 velocity=11.6 -> lower=-2.5394 upper=2.5546 effort=55.0 velocity=11.72; origin xyz=-0.015 0.05615 -0.061 -> xyz=-0.015 0.05515 -0.095
- joint j_arm2_6: axis 0 -1 0 -> 0 1 0; limit lower=-1.4726 upper=1.5364 effort=55 velocity=11.6 -> lower=-1.5154 upper=1.5156 effort=55.0 velocity=11.72; origin xyz=0.0 -0.049 -0.18 -> xyz=0.0 -0.049 -0.156
- joint j_arm2_7: axis 0 0 -1 -> 0 0 1; limit lower=-3.0908 upper=2.0114 effort=27 velocity=20.3 -> lower=-2.5554 upper=2.5686 effort=28.32 velocity=20.35; origin xyz=0.0 0.049 -0.169 -> xyz=0.0 0.049 -0.174
- joint j_arm2_8: origin xyz=0.0 0.0 -0.0405 rpy=0.0 3.14159265359 -1.5707963268 -> xyz=0.0 0.0 -0.035 rpy=0.0 3.14159265359 0.0; parent arm2_7 -> ft_arm2
- joint j_kinect_optical_frame: origin xyz=0.050 -0.110 -0.035 rpy= -1.5707963268 0 -1.5707963268 -> rpy= -1.5707963268 0 -1.5707963268; parent kinect -> kinect2_rgb_frame
- joint j_velodyne: origin xyz=-0.138 0.0 -0.033 rpy=0.0 0.0 -3.14159265359 -> xyz=0.0283656 -0.00976704 0.047 rpy=1.57079632679 0.0 -0.331612273666
- joint neck_pitch: limit lower=-0.34906585 upper=1.4 effort=35 velocity=5.7 -> lower=-0.34906585 upper=0.78539816 effort=35 velocity=5.7

File: configs/mwoibn/urdf/centauro_lower_body.urdf (robot description, URDF)
Before this commit: robot centauro, 27 links, 26 joints
Links:
- link pelvis: mass 24.190945 -> 16.097574
Joints:
- joint hip_yaw_1: limit lower=-0.9432 upper=2.5138 effort=304 velocity=8.8 -> lower=-2.03 upper=1.2 effort=304 velocity=8.8
- joint hip_yaw_2: limit lower=-2.511 upper=0.943 effort=304 velocity=8.8 -> lower=-1.2 upper=2.03 effort=304 velocity=8.8
- joint hip_yaw_3: limit lower=-2.51 upper=0.943 effort=304 velocity=8.8 -> lower=-1.2 upper=2.03 effort=304 velocity=8.8
- joint hip_yaw_4: limit lower=-0.9412 upper=2.5138 effort=304 velocity=8.8 -> lower=-2.03 upper=1.2 effort=304 velocity=8.8
- joint imu_joint: origin xyz=0.0 0.0 0.0 rpy=0.0 0.0 0.0 -> xyz=0.248316 0.0 0.015 rpy=0.0 0.0 0.0

File: configs/mwoibn/urdf/centauro_upper_body.urdf (robot description, URDF)
Before this commit: robot centauro, 28 links, 27 joints
Links:
- added link ft_arm1, mass 0.37827821; collision mesh filename=package://centauro/centauro_urdf/meshes/convex_hull/link9.s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 scale=0.001 -0.001 0.001; visual mesh filename=package://centauro/centauro_urdf/meshes/simplified/Wrist.STL scale=0.001 -0.001 0.001
- added link ft_arm2, mass 0.37827821; collision mesh filename=package://centauro/centauro_urdf/meshes/convex_hull/link9.s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 scale=0.001 0.001 0.001; visual mesh filename=package://centauro/centauro_urdf/meshes/simplified/Wrist.STL scale=0.001 0.001 0.001
- added link kinect2_rgb_frame
- added link velodyne_calib
- link arm1_1: mass 1.5583338 -> 1.9628675; geometry collision mesh filename=package://centauro/centauro_urdf/meshes/convex_hull/link2.s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 scale=0.001 -0.001 0.001; visual mesh filename=package://centauro/centauro_urdf/meshes/simplified/Shoulder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 scale=0.001 -0.001 0.001
- link arm1_2: mass 1.515061 -> 1.8595811; geometry collision mesh filename=package://centauro/centauro_urdf/meshes/convex_hull/link3.s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 scale=0.001 -0.001 0.001; visual mesh filename=package://centauro/centauro_urdf/meshes/simplified/Shoulder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 scale=0.001 -0.001 0.001
- link arm1_3: mass 1.5088101 -> 1.6678109; geometry collision mesh filename=package://centauro/centauro_urdf/meshes/convex_hull/link4.s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 scale=0.001 -0.001 0.001; visual mesh filename=package://centauro/centauro_urdf/meshes/simplified/Shoulder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 scale=0.001 -0.001 0.001
- link arm1_4: mass 0.96297329 -> 1.3157289; geometry collision mesh filename=package://centauro/centauro_urdf/meshes/convex_hull/link5.s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 scale=0.001 -0.001 0.001; visual mesh filename=package://centauro/centauro_urdf/meshes/simplified/Elbow.STL scale=0.001 -0.001 0.001
- link arm1_5: mass 1.4703698 -> 1.4908547; geometry collision mesh filename=package://centauro/centauro_urdf/meshes/convex_hull/link6.s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 scale=0.001 -0.001 0.001; visual mesh filename=package://centauro/centauro_urdf/meshes/simplified/Forearm.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 scale=0.001 -0.001 0.001
- link arm1_6: mass 0.94693868 -> 1.1263612; geometry collision mesh filename=package://centauro/centauro_urdf/meshes/convex_hull/link7.s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 scale=0.001 -0.001 0.001; visual mesh filename=package://centauro/centauro_urdf/meshes/simplified/ForearmP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 scale=0.001 -0.001 0.001
- link arm1_7: mass 0.55981036 -> 0.27966428; geometry collision mesh filename=package://centauro/centauro_urdf/meshes/convex_hull/link8.s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 scale=0.001 -0.001 0.001; visual mesh filename=package://centauro/centauro_urdf/meshes/simplified/ForearmY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 scale=0.001 -0.001 0.001
- link arm1_8: mass 0.15 -> 1.8366865; geometry collision mesh filename=package://centauro/centauro_urdf/meshes/convex_hull/heri.stl scale=0.001 -0.001 -0.001; visual mesh filename=package://centauro/centauro_urdf/meshes/simplified/heri.stl scale=0.001 -0.001 -0.001
- link arm2_1: mass 1.5583338 -> 1.9628675; geometry collision mesh filename=package://centauro/centauro_urdf/meshes/convex_hull/link2.s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 scale=0.001 0.001 0.001; visual mesh filename=package://centauro/centauro_urdf/meshes/simplified/Shoulder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 scale=0.001 0.001 0.001
- link arm2_2: mass 1.515061 -> 1.8595811; geometry collision mesh filename=package://centauro/centauro_urdf/meshes/convex_hull/link3.s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 scale=0.001 0.001 0.001; visual mesh filename=package://centauro/centauro_urdf/meshes/simplified/Shoulder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 scale=0.001 0.001 0.001
- link arm2_3: mass 1.5088101 -> 1.6678109; geometry collision mesh filename=package://centauro/centauro_urdf/meshes/convex_hull/link4.s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 scale=0.001 0.001 0.001; visual mesh filename=package://centauro/centauro_urdf/meshes/simplified/Shoulder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 scale=0.001 0.001 0.001
- link arm2_4: mass 0.96297329 -> 1.3157289; geometry collision mesh filename=package://centauro/centauro_urdf/meshes/convex_hull/link5.s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 scale=0.001 0.001 0.001; visual mesh filename=package://centauro/centauro_urdf/meshes/simplified/Elbow.STL scale=0.001 0.001 0.001
- link arm2_5: mass 1.4703698 -> 1.4908547; geometry collision mesh filename=package://centauro/centauro_urdf/meshes/convex_hull/link6.s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 scale=0.001 0.001 0.001; visual mesh filename=package://centauro/centauro_urdf/meshes/simplified/Forearm.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 scale=0.001 0.001 0.001
- link arm2_6: mass 0.94693868 -> 1.1263612; geometry collision mesh filename=package://centauro/centauro_urdf/meshes/convex_hull/link7.s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 scale=0.001 0.001 0.001; visual mesh filename=package://centauro/centauro_urdf/meshes/simplified/ForearmP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 scale=0.001 0.001 0.001
- link arm2_7: mass 0.55981036 -> 0.27966428; geometry collision mesh filename=package://centauro/centauro_urdf/meshes/convex_hull/link8.s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 scale=0.001 0.001 0.001; visual mesh filename=package://centauro/centauro_urdf/meshes/simplified/ForearmY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 scale=0.001 0.001 0.001
- link neck_3: geometry collision mesh filename=package://centauro/centauro_urdf/meshes/convex_hull/velodyn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 scale=0.001 0.001 0.001; visual mesh filename=package://centauro/centauro_urdf/meshes/simplified/mesh_lid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 scale=0.001 0.001 0.001
- link torso_2: mass 6.1886404 -> 11.492689
Joints:
- added joint j_ft_1: type fixed, parent arm1_7, child ft_arm1, origin xyz=0.0 0.0 -0.0 rpy=0.0 0.0 0.0, axis 0 0 1, limit lower=0.0 upper=0.0 effort=0 velocity=0
- added joint j_ft_2: type fixed, parent arm2_7, child ft_arm2, origin xyz=0.0 0.0 -0.0 rpy=0.0 0.0 0.0, axis 0 0 1, limit lower=0.0 upper=0.0 effort=0 velocity=0
- added joint j_kinect2_rgb_frame: type fixed, parent kinect, child kinect2_rgb_frame, origin xyz=0.050 -0.110 -0.035
- added joint velodyne_calib: type fixed, parent neck_3, child velodyne_calib, origin xyz=-0.175768 0 -0.034219 rpy=-1.57772 0.0128311 1.57073
- joint j_arm1_1: axis 0 0.984807753012 0.173648177667 -> 0 1 0; limit lower=-3.348 upper=1.578 effort=147 velocity=5.7 -> lower=-3.312 upper=1.615 effort=147.0 velocity=3.86; origin xyz=0.04576 0.169137 0.116626 rpy=0.0 0.0 -0.523602668986 -> xyz=0.0457475 0.169137 0.116626 rpy=0.174533 0.0 -0.5235988
- joint j_arm1_2: axis -1 0 0 -> 1 0 0; limit lower=-3.42 upper=-0.056 effort=147 velocity=5.7 -> lower=0.02 upper=3.431 effort=147.0 velocity=3.86; origin xyz=-0.09115 0.06106 0.010766 -> xyz=-0.09015 0.062 0.0 rpy=-0.1745327 0.0 0.0
- joint j_arm1_3: axis 0 0 -1 -> 0 0 1; limit lower=-2.5556 upper=2.5424 effort=147 velocity=8.2 -> lower=-2.552 upper=2.566 effort=147.0 velocity=6.06; origin xyz=0.09115 0.0 -0.21915 -> xyz=0.09015 0.0 -0.21815
- joint j_arm1_4: limit lower=-2.4636 upper=0.2804 effort=147 velocity=8.2 -> lower=-2.465 upper=0.28 effort=147.0 velocity=6.06; origin xyz=0.04 0.05615 -0.074 -> xyz=0.045 0.05515 -0.074
- joint j_arm1_5: axis 0 0 -1 -> 0 0 1; limit lower=-2.5406 upper=2.5534 effort=55 velocity=11.6 -> lower=-2.569 upper=2.562 effort=55.0 velocity=11.72; origin xyz=-0.015 -0.05615 -0.061 -> xyz=-0.015 -0.05515 -0.095
- joint j_arm1_6: limit lower=-1.5096 upper=1.5044 effort=55 velocity=11.6 -> lower=-1.529 upper=1.509 effort=55.0 velocity=11.72; origin xyz=0.0 0.049 -0.18 -> xyz=0.0 0.049 -0.156
- joint j_arm1_7: axis 0 0 -1 -> 0 0 1; limit lower=-2.5376 upper=2.5554 effort=27 velocity=20.3 -> lower=-2.565 upper=2.569 effort=28.32 velocity=20.35; origin xyz=0.0 -0.049 -0.169 -> xyz=0.0 -0.049 -0.174
- joint j_arm1_8: origin xyz=0.0 0.0 -0.0405 rpy=0.0 3.14159265359 -1.5707963268 -> xyz=0.0 0.0 -0.0415 rpy=0.0 3.14159265359 3.14159265359; parent arm1_7 -> ft_arm1
- joint j_arm2_1: axis 0 -0.984807753012 0.173648177667 -> 0 1 0; limit lower=-1.6102 upper=3.3138 effort=147 velocity=5.7 -> lower=-3.3458 upper=1.6012 effort=147.0 velocity=3.86; origin xyz=0.04576 -0.169137 0.116626 rpy=0.0 0.0 0.523602668986 -> xyz=0.0457475 -0.169137 0.116626 rpy=0.174533 0.0 0.5235988
- joint j_arm2_2: axis -1 0 0 -> 1 0 0; limit lower=0.0578 upper=3.4288 effort=147 velocity=5.7 -> lower=-3.4258 upper=-0.0138 effort=147.0 velocity=3.86; origin xyz=-0.09115 -0.06106 0.010766 -> xyz=-0.09015 -0.062 0.0 rpy=-0.1745327 0.0 0.0
- joint j_arm2_3: axis 0 0 -1 -> 0 0 1; limit lower=-2.5426 upper=2.5524 effort=147 velocity=8.2 -> lower=-2.5614 upper=2.5606 effort=147.0 velocity=6.06; origin xyz=0.09115 0.0 -0.21915 -> xyz=0.09015 0.0 -0.21815
- joint j_arm2_4: axis 0 -1 0 -> 0 1 0; limit lower=-0.2796 upper=2.4564 effort=147 velocity=8.2 -> lower=-2.4794 upper=0.2886 effort=147.0 velocity=6.06; origin xyz=0.04 -0.05615 -0.074 -> xyz=0.045 -0.05515 -0.074
- joint j_arm2_5: axis 0 0 -1 -> 0 0 1; limit lower=-2.5626 upper=2.5464 effort=55 velocity=11.6 -> lower=-2.5394 upper=2.5546 effort=55.0 velocity=11.72; origin xyz=-0.015 0.05615 -0.061 -> xyz=-0.015 0.05515 -0.095
- joint j_arm2_6: axis 0 -1 0 -> 0 1 0; limit lower=-1.4726 upper=1.5364 effort=55 velocity=11.6 -> lower=-1.5154 upper=1.5156 effort=55.0 velocity=11.72; origin xyz=0.0 -0.049 -0.18 -> xyz=0.0 -0.049 -0.156
- joint j_arm2_7: axis 0 0 -1 -> 0 0 1; limit lower=-3.0908 upper=2.0114 effort=27 velocity=20.3 -> lower=-2.5554 upper=2.5686 effort=28.32 velocity=20.35; origin xyz=0.0 0.049 -0.169 -> xyz=0.0 0.049 -0.174
- joint j_arm2_8: origin xyz=0.0 0.0 -0.0405 rpy=0.0 3.14159265359 -1.5707963268 -> xyz=0.0 0.0 -0.035 rpy=0.0 3.14159265359 0.0; parent arm2_7 -> ft_arm2
- joint j_kinect_optical_frame: origin xyz=0.050 -0.110 -0.035 rpy= -1.5707963268 0 -1.5707963268 -> rpy= -1.5707963268 0 -1.5707963268; parent kinect -> kinect2_rgb_frame
- joint j_velodyne: origin xyz=-0.138 0.0 -0.033 rpy=0.0 0.0 -3.14159265359 -> xyz=0.0283656 -0.00976704 0.047 rpy=1.57079632679 0.0 -0.331612273666
