Commit message: XBot URDF limits update, Misc experimens changes: logged data

File: configs/mwoibn/urdf/centauro.urdf (robot description, URDF)
Before this commit: robot centauro, 57 links, 56 joints
Joints:
- joint ankle_pitch_1: limit lower=-2.4056 upper=2.3184 effort=147 velocity=8.1 -> lower=-2.4056 upper=2.3184 effort=98 velocity=1.0
- joint ankle_pitch_2: limit lower=-2.3266 upper=2.3914 effort=147 velocity=8.1 -> lower=-2.3266 upper=2.3914 effort=98 velocity=1.0
- joint ankle_pitch_3: limit lower=-2.4696 upper=2.4464 effort=147 velocity=8.1 -> lower=-2.4696 upper=2.4464 effort=98 velocity=1.0
- joint ankle_pitch_4: limit lower=-2.3426 upper=2.3934 effort=147 velocity=8.1 -> lower=-2.3426 upper=2.3934 effort=98 velocity=1.0
- joint ankle_yaw_1: limit lower=-2.5626 upper=2.5384 effort=35 velocity=20.0 -> lower=-2.5626 upper=2.5384 effort=23 velocity=1.0
- joint ankle_yaw_2: limit lower=-2.5546 upper=2.5484 effort=35 velocity=20.0 -> lower=-2.5546 upper=2.5484 effort=23 velocity=1.0
- joint ankle_yaw_3: limit lower=-2.5606 upper=2.5454 effort=35 velocity=20.0 -> lower=-2.5606 upper=2.5454 effort=23 velocity=1.0
- joint ankle_yaw_4: limit lower=-2.6046 upper=2.5514 effort=35 velocity=20.0 -> lower=-2.6046 upper=2.5514 effort=23 velocity=1.0
- joint hip_pitch_1: limit lower=-2.0226 upper=2.02748 effort=304 velocity=8.8 -> lower=-2.0226 upper=2.02748 effort=200 velocity=1.0
- joint hip_pitch_2: limit lower=-2.0156 upper=2.0354 effort=304 velocity=8.8 -> lower=-2.0156 upper=2.0354 effort=200 velocity=1.0
- joint hip_pitch_3: limit lower=-2.0126 upper=2.0384 effort=304 velocity=8.8 -> lower=-2.0126 upper=2.0384 effort=200 velocity=1.0
- joint hip_pitch_4: limit lower=-2.0326 upper=2.0524 effort=304 velocity=8.8 -> lower=-2.0326 upper=2.0524 effort=200 velocity=1.0
- joint hip_yaw_1: limit lower=-2.03 upper=1.2 effort=304 velocity=8.8 -> lower=-2.03 upper=1.2 effort=200 velocity=1.0
- joint hip_yaw_2: limit lower=-1.2 upper=2.03 effort=304 velocity=8.8 -> lower=-1.2 upper=2.03 effort=200 velocity=1.0
- joint hip_yaw_3: limit lower=-1.2 upper=2.03 effort=304 velocity=8.8 -> lower=-1.2 upper=2.03 effort=200 velocity=1.0
- joint hip_yaw_4: limit lower=-2.03 upper=1.2 effort=304 velocity=8.8 -> lower=-2.03 upper=1.2 effort=200 velocity=1.0
- joint j_wheel_1: limit effort=35 velocity=20.0 -> effort=23 velocity=1.0
- joint j_wheel_2: limit effort=35 velocity=20.0 -> effort=23 velocity=1.0
- joint j_wheel_3: limit effort=35 velocity=20.0 -> effort=23 velocity=1.0
- joint j_wheel_4: limit effort=35 velocity=20.0 -> effort=23 velocity=1.0
- joint knee_pitch_1: limit lower=-2.4056 upper=2.3994 effort=304 velocity=8.8 -> lower=-2.4056 upper=2.3994 effort=200 velocity=1.0
- joint knee_pitch_2: limit lower=-2.4006 upper=2.4034 effort=304 velocity=8.8 -> lower=-2.4006 upper=2.4034 effort=200 velocity=1.0
- joint knee_pitch_3: limit lower=-2.4056 upper=2.4064 effort=304 velocity=8.8 -> lower=-2.4056 upper=2.4064 effort=200 velocity=1.0
- joint knee_pitch_4: limit lower=-2.4176 upper=2.3884 effort=304 velocity=8.8 -> lower=-2.4176 upper=2.3884 effort=200 velocity=1.0

File: configs/mwoibn/urdf/centauro_lower_body.urdf (robot description, URDF)
Before this commit: robot centauro, 27 links, 26 joints
Joints:
- joint ankle_pitch_1: limit lower=-2.4056 upper=2.3184 effort=147 velocity=8.1 -> lower=-2.4056 upper=2.3184 effort=98 velocity=1.0
- joint ankle_pitch_2: limit lower=-2.3266 upper=2.3914 effort=147 velocity=8.1 -> lower=-2.3266 upper=2.3914 effort=98 velocity=1.0
- joint ankle_pitch_3: limit lower=-2.4696 upper=2.4464 effort=147 velocity=8.1 -> lower=-2.4696 upper=2.4464 effort=98 velocity=1.0
- joint ankle_pitch_4: limit lower=-2.3426 upper=2.3934 effort=147 velocity=8.1 -> lower=-2.3426 upper=2.3934 effort=98 velocity=1.0
- joint ankle_yaw_1: limit lower=-2.5626 upper=2.5384 effort=35 velocity=20.0 -> lower=-2.5626 upper=2.5384 effort=23 velocity=1.0
- joint ankle_yaw_2: limit lower=-2.5546 upper=2.5484 effort=35 velocity=20.0 -> lower=-2.5546 upper=2.5484 effort=23 velocity=1.0
- joint ankle_yaw_3: limit lower=-2.5606 upper=2.5454 effort=35 velocity=20.0 -> lower=-2.5606 upper=2.5454 effort=23 velocity=1.0
- joint ankle_yaw_4: limit lower=-2.6046 upper=2.5514 effort=35 velocity=20.0 -> lower=-2.6046 upper=2.5514 effort=23 velocity=1.0
- joint hip_pitch_1: limit lower=-2.0226 upper=2.02748 effort=304 velocity=8.8 -> lower=-2.0226 upper=2.02748 effort=200 velocity=1.0
- joint hip_pitch_2: limit lower=-2.0156 upper=2.0354 effort=304 velocity=8.8 -> lower=-2.0156 upper=2.0354 effort=200 velocity=1.0
- joint hip_pitch_3: limit lower=-2.0126 upper=2.0384 effort=304 velocity=8.8 -> lower=-2.0126 upper=2.0384 effort=200 velocity=1.0
- joint hip_pitch_4: limit lower=-2.0326 upper=2.0524 effort=304 velocity=8.8 -> lower=-2.0326 upper=2.0524 effort=200 velocity=1.0
- joint hip_yaw_1: limit lower=-2.03 upper=1.2 effort=304 velocity=8.8 -> lower=-2.03 upper=1.2 effort=200 velocity=1.0
- joint hip_yaw_2: limit lower=-1.2 upper=2.03 effort=304 velocity=8.8 -> lower=-1.2 upper=2.03 effort=200 velocity=1.0
- joint hip_yaw_3: limit lower=-1.2 upper=2.03 effort=304 velocity=8.8 -> lower=-1.2 upper=2.03 effort=200 velocity=1.0
- joint hip_yaw_4: limit lower=-2.03 upper=1.2 effort=304 velocity=8.8 -> lower=-2.03 upper=1.2 effort=200 velocity=1.0
- joint j_wheel_1: limit effort=35 velocity=20.0 -> effort=23 velocity=1.0
- joint j_wheel_2: limit effort=35 velocity=20.0 -> effort=23 velocity=1.0
- joint j_wheel_3: limit effort=35 velocity=20.0 -> effort=23 velocity=1.0
- joint j_wheel_4: limit effort=35 velocity=20.0 -> effort=23 velocity=1.0
- joint knee_pitch_1: limit lower=-2.4056 upper=2.3994 effort=304 velocity=8.8 -> lower=-2.4056 upper=2.3994 effort=200 velocity=1.0
- joint knee_pitch_2: limit lower=-2.4006 upper=2.4034 effort=304 velocity=8.8 -> lower=-2.4006 upper=2.4034 effort=200 velocity=1.0
- joint knee_pitch_3: limit lower=-2.4056 upper=2.4064 effort=304 velocity=8.8 -> lower=-2.4056 upper=2.4064 effort=200 velocity=1.0
- joint knee_pitch_4: limit lower=-2.4176 upper=2.3884 effort=304 velocity=8.8 -> lower=-2.4176 upper=2.3884 effort=200 velocity=1.0

Commit message: correct odometry initialization issue

File: configs/mwoibn/urdf/centauro.urdf (robot description, URDF)
Before this commit: robot centauro, 57 links, 56 joints
Joints:
- joint ankle_yaw_1: limit lower=-2.5626 upper=2.5384 effort=23 velocity=1.0 -> lower=-2.5626 upper=2.5384 effort=23 velocity=2.0
- joint ankle_yaw_2: limit lower=-2.5546 upper=2.5484 effort=23 velocity=1.0 -> lower=-2.5546 upper=2.5484 effort=23 velocity=2.0
- joint ankle_yaw_3: limit lower=-2.5606 upper=2.5454 effort=23 velocity=1.0 -> lower=-2.5606 upper=2.5454 effort=23 velocity=2.0
- joint ankle_yaw_4: limit lower=-2.6046 upper=2.5514 effort=23 velocity=1.0 -> lower=-2.6046 upper=2.5514 effort=23 velocity=2.0
- joint j_wheel_1: limit effort=23 velocity=1.0 -> effort=23 velocity=2.0
- joint j_wheel_2: limit effort=23 velocity=1.0 -> effort=23 velocity=2.0
- joint j_wheel_3: limit effort=23 velocity=1.0 -> effort=23 velocity=2.0
- joint j_wheel_4: limit effort=23 velocity=1.0 -> effort=23 velocity=2.0

Commit message: experiments updates * XBot long names * config tunning * steering saturation

File: configs/mwoibn/urdf/centauro.urdf (robot description, URDF)
Before this commit: robot centauro, 57 links, 56 joints
Joints:
- joint ankle_yaw_1: limit lower=-2.5626 upper=2.5384 effort=23 velocity=2.0 -> lower=-2.5626 upper=2.5384 effort=23 velocity=1.0
- joint ankle_yaw_2: limit lower=-2.5546 upper=2.5484 effort=23 velocity=2.0 -> lower=-2.5546 upper=2.5484 effort=23 velocity=1.0
- joint ankle_yaw_3: limit lower=-2.5606 upper=2.5454 effort=23 velocity=2.0 -> lower=-2.5606 upper=2.5454 effort=23 velocity=1.0
- joint ankle_yaw_4: limit lower=-2.6046 upper=2.5514 effort=23 velocity=2.0 -> lower=-2.6046 upper=2.5514 effort=23 velocity=1.0
- joint j_wheel_1: limit effort=23 velocity=2.0 -> effort=23 velocity=1.0
- joint j_wheel_2: limit effort=23 velocity=2.0 -> effort=23 velocity=1.0
- joint j_wheel_3: limit effort=23 velocity=2.0 -> effort=23 velocity=1.0
- joint j_wheel_4: limit effort=23 velocity=2.0 -> effort=23 velocity=1.0
